Commit message: Agregar plano eléctrico rev. 1.0 y su documentación
- Plano de Mesa de Cableado (37 componentes, 137 cables)
- Tabla de cableado generada desde el plano + script para regenerarla
- Presupuesto de potencia con autonomía estimada
- Árbol de potencia y señales de control en el README de esquemáticos
- Revisión del plano con 17 puntos pendientes
- Radio de rueda real (6.5") en el URDF

Co-Authored-By: Claude Opus 5.5 <noreply@anthropic.com>
Claude-Session: https://claude.ai/code/session_01BTW9ot9YC3wLhXhE3iwN4N

File: milo_description/urdf/milo.urdf.xacro (robot description, xacro)
@@ -15,5 +15,5 @@
   <xacro:property name="base_mass"     value="20.0"/>
   <xacro:property name="base_z"        value="0.05"/>   <!-- altura del fondo del chasis sobre el suelo -->
-  <xacro:property name="wheel_radius"  value="0.08"/>
+  <xacro:property name="wheel_radius"  value="0.0826"/> <!-- rueda de hoverboard 6.5" (dato real) -->
   <xacro:property name="wheel_width"   value="0.04"/>
   <xacro:property name="wheel_mass"    value="1.0"/>
